File: high-current-sense-relay.sch (KiCad schematic (older format))
At the start: 15 parts, among them J1 Conn_01x01_Female, J2 Conn_01x01_Female, J3 Conn_01x04_Male, U1 ATtiny85-20PU, U2 OPAMP, U3 ACS758xCB-150B-PFF

Commit message: intr
Parts:
- removed U2: OPAMP, symbol pspice:OPAMP
- added U2: MCP6001U, high-current-sense-relay:SOT95P280X145-5N, symbol Amplifier_Operational:MCP6001U
- C1, C2: footprint (none) -> high-current-sense-relay:K104K15X7RF53H5
- D1: footprint (none) -> high-current-sense-relay:DIO_1N4447
- D2, D3: footprint (none) -> high-current-sense-relay:LTL4232
- J1, J2: footprint (none) -> high-current-sense-relay:LAMA6-14QY
- J3: footprint (none) -> Connector_PinHeader_2.54mm:PinHeader_1x04_P2.54mm_Vertical
- R1: value R -> 47k; footprint (none) -> Resistor_THT:R_Axial_DIN0204_L3.6mm_D1.6mm_P7.62mm_Horizontal
- R2: value R -> 3k; footprint (none) -> Resistor_THT:R_Axial_DIN0204_L3.6mm_D1.6mm_P1.90mm_Vertical
- R3, R4: footprint (none) -> Resistor_THT:R_Axial_DIN0204_L3.6mm_D1.6mm_P1.90mm_Vertical
Connections:
- net +3.3V is gone; now on net +3V3: C1.1, C2.1, D1.1 (K), R3.1, U1.8 (VCC), U3.1 (VCC)
- net +3V3: now also U2.5 (V+)
- net GND: now also U2.2 (V-)
- net IP+: now also R2.2
- net IP-: now also R1.1
- net VSense: now also U2.1 (+), U2.4
- net at D1.2 (A), R1.2, R2.1: now also U2.3 (-)
- no-connect marks 0 -> 1
Other:
- moved on the sheet: C1, U1
